File: ECMag.sch (KiCad schematic (older format))
At the start: 40 parts, among them J1 Conn_01x12_Male, J2 Conn_01x05_Male, J3 Conn_01x04_Male, J4 USB_B, K1 NA, K2 NA, K3 NA, K4 NA, P1 10K, Q1 BC548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

Commit message: Esquemáticounifilar terminado. Faltan footprints y datasheets
Parts:
- removed J1: Conn_01x12_Male, symbol Connector:Conn_01x12_Male
- removed J2: Conn_01x05_Male, symbol Connector:Conn_01x05_Male
- removed J3: Conn_01x04_Male, symbol Connector:Conn_01x04_Male
- removed J4: USB_B, symbol Connector:USB_B
- added J1: Conn_01x12, symbol Connector_Generic:Conn_01x12
- added J2: Conn_01x05, symbol Connector_Generic:Conn_01x05
- added J3, J6: Conn_01x04, symbol Connector_Generic:Conn_01x04
- added J4: USB_B, symbol Enc_Mag:USB_B
- added J5: Barrel_Jack_SW, symbol Connector:Barrel_Jack_Switch
- renumbered D4 to D2, D2 to D3, D3 to D4
Connections:
- net labels added: D+, D-, RxSgn, TxSgn
- wire segments 141 -> 160
- no-connect marks 17 -> 18
Other:
- note added: "Conector Encoder"
- note added: "Conectores Sensor Mag. Display e Inalambrico"
- note added: "Ficha de Alimentación, Ficha USB y leds Rx Tx y Pwr"
- note removed: "Conectores Externos"
- moved on the sheet: BZ1, C1, C10, C11, C2, C3, C4, C5, C6, C7, C8, C9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

Commit message: Esquemático terminado, con footprints y datasheets
Parts:
- added R10: 3K3 5%, Resistor_THT:R_Axial_DIN0207_L6.3mm_D2.5mm_P7.62mm_Horizontal, symbol Enc_Mag:Resistencia
- BZ1: value Buzzer -> Buzzer 5V 85db 2300Hz; footprint (none) -> Buzzer_Beeper:Buzzer_12x9.5RM7.6
- C1, C3: value 220uF -> 220uF 25v HT; footprint (none) -> Capacitor_THT:CP_Radial_D8.0mm_P5.00mm
- C10, C9: value 1uF -> 100nF; footprint (none) -> Capacitor_THT:C_Disc_D5.1mm_W3.2mm_P5.00mm
- C11: footprint (none) -> Capacitor_THT:C_Disc_D5.1mm_W3.2mm_P5.00mm
- C2, C4: value 100nF -> 100nF Cerámico; footprint (none) -> Capacitor_THT:C_Disc_D5.1mm_W3.2mm_P5.00mm
- C5, C6, C7, C8: footprint (none) -> Capacitor_THT:C_Disc_D6.0mm_W2.5mm_P5.00mm
- D1: value SS14 -> 1N5822; footprint (none) -> Diode_THT:D_DO-27_P15.24mm_Horizontal
- D2, D3, D4: footprint (none) -> LED_THT:LED_D3.0mm
- J4: footprint (none) -> Connector_USB:USB_B_OST_USB-B1HSxx_Horizontal
- J5: footprint (none) -> Connector_BarrelJack:BarrelJack_Wuerth_6941xx301002
- K1, K2, K3, K4: value NA -> Tactil Switch B3F NA; footprint (none) -> Button_Switch_THT:SW_PUSH_6mm_H5mm
- L1: footprint (none) -> Inductor_THT:L_Radial_D7.5mm_P5.00mm_Fastron_07P
- P1: footprint (none) -> Potentiometer_THT:Potentiometer_Bourns_3266W_Vertical
- R1: value 330 -> 330 1%; footprint (none) -> Resistor_THT:R_Axial_DIN0207_L6.3mm_D2.5mm_P7.62mm_Horizontal
- R2, R3, R4, R5: value 10K -> 10K 5%; footprint (none) -> Resistor_THT:R_Axial_DIN0207_L6.3mm_D2.5mm_P7.62mm_Horizontal
- R6, R7, R8: value 4K7 -> 4K7 5%; footprint (none) -> Resistor_THT:R_Axial_DIN0207_L6.3mm_D2.5mm_P7.62mm_Horizontal
- U3: footprint (none) -> Package_TO_SOT_SMD:TO-263-5_TabPin6
- Y1: value 20HHz -> 16MHz; footprint (none) -> Crystal:Crystal_HC49-U_Vertical
- Y2: value 16MHz -> 20MHz; footprint (none) -> Crystal:Crystal_HC49-U_Vertical
Connections:
- net BZZ: now also R10.1; no longer Q1.2 (B)
- new net: Q1.2 (B), R10.2
Other:
- note added: "Conectores Sensor Magnético Display e Inalambrico"
- note removed: "Conectores Sensor Mag. Display e Inalambrico"
- moved on the sheet: C1, C2, P1, R1
